Commit message: Add calibration world and tune wheel separation

File: src/brover_simulation/urdf/brover_e5.urdf.xacro (robot description, xacro)
@@ -28,5 +28,5 @@
   <xacro:property name="wheel_width" value="0.065"/>
   <xacro:property name="wheel_y" value="0.2132"/>
-  <xacro:property name="wheel_separation" value="0.4264"/>
+  <xacro:property name="wheel_separation" value="0.58"/>
   <xacro:property name="wheel_z" value="-0.080"/>
   <xacro:property name="front_wheel_x" value="0.210"/>

Commit message: Tune lidar scan orientation

File: src/brover_simulation/urdf/brover_e5.urdf.xacro (robot description, xacro)
@@ -28,5 +28,5 @@
   <xacro:property name="wheel_width" value="0.065"/>
   <xacro:property name="wheel_y" value="0.2132"/>
-  <xacro:property name="wheel_separation" value="0.58"/>
+  <xacro:property name="wheel_separation" value="0.572"/>
   <xacro:property name="wheel_z" value="-0.080"/>
   <xacro:property name="front_wheel_x" value="0.210"/>
@@ -169,5 +169,5 @@
     <parent link="base_link"/>
     <child link="lidar_link"/>
-    <origin xyz="0.113 0 0.149" rpy="0 0 0"/>
+    <origin xyz="0.113 0 0.149" rpy="0 0 3.141592653589793"/>
   </joint>
   <link name="front_camera_link"/>
